Commit message: Change turtlebot sensor naming for consistency

File: robots/kobuki_hexagons_toto.urdf.xacro (robot description, xacro)
@@ -16,43 +16,41 @@
   <sensor_kinect  parent="base_link"/> <!--add sensors-->
   <!--Add custom sensors-->
-  <!--TEMPLATE
-  <xacro:sonar_sensor name="sonar" parent="base_link" ros_topic="sonar_height" update_rate="10" min_range="0.01" max_range="3.0" field_of_view="${40*M_PI/180}" ray_count="3">
-    <origin xyz="0 0.0 0.42" rpy="0 0 0"/>
-  </xacro:sonar_sensor>
-  -->
-  <xacro:sonar_sensor name="sonar_sensor_zero" parent="base_link" ros_topic="sonar_zero" update_rate="10" min_range="0.01" max_range="3.0" field_of_view="${30*M_PI/180}" ray_count="3">
+  <!--Magnetometer/compass-->
+  <!--TODO: Add compass-->
+  <!-- Sonars -->
+  <xacro:sonar_sensor name="sonar_sensor_zero" parent="base_link" ros_topic="sonar_0" update_rate="10" min_range="0.01" max_range="2.55" field_of_view="${30*M_PI/180}" ray_count="3">
     <origin xyz="0.0 0.0 ${SONAR_HEIGHT}" rpy="0 0 1.309"/>
   </xacro:sonar_sensor>
-  <xacro:sonar_sensor name="sonar_sensor_one" parent="base_link" ros_topic="sonar_one" update_rate="10" min_range="0.01" max_range="3.0" field_of_view="${30*M_PI/180}" ray_count="3">
+  <xacro:sonar_sensor name="sonar_sensor_one" parent="base_link" ros_topic="sonar_1" update_rate="10" min_range="0.01" max_range="2.55" field_of_view="${30*M_PI/180}" ray_count="3">
     <origin xyz="0.00 0.0 ${SONAR_HEIGHT}" rpy="0 0 0.785"/>
   </xacro:sonar_sensor>
-  <xacro:sonar_sensor name="sonar_sensor_two" parent="base_link" ros_topic="sonar_two" update_rate="10" min_range="0.01" max_range="3.0" field_of_view="${30*M_PI/180}" ray_count="3">
+  <xacro:sonar_sensor name="sonar_sensor_two" parent="base_link" ros_topic="sonar_2" update_rate="10" min_range="0.01" max_range="2.55" field_of_view="${30*M_PI/180}" ray_count="3">
     <origin xyz="0.0 0.0 ${SONAR_HEIGHT}" rpy="0 0 0.262"/>
   </xacro:sonar_sensor>
-  <xacro:sonar_sensor name="sonar_sensor_three" parent="base_link" ros_topic="sonar_three" update_rate="10" min_range="0.01" max_range="3.0" field_of_view="${30*M_PI/180}" ray_count="3">
+  <xacro:sonar_sensor name="sonar_sensor_three" parent="base_link" ros_topic="sonar_3" update_rate="10" min_range="0.01" max_range="2.55" field_of_view="${30*M_PI/180}" ray_count="3">
     <origin xyz="0.0 0.0 ${SONAR_HEIGHT}" rpy="0 0 -0.262"/>
   </xacro:sonar_sensor>
-  <xacro:sonar_sensor name="sonar_sensor_four" parent="base_link" ros_topic="sonar_four" update_rate="10" min_range="0.01" max_range="3.0" field_of_view="${30*M_PI/180}" ray_count="3">
+  <xacro:sonar_sensor name="sonar_sensor_four" parent="base_link" ros_topic="sonar_4" update_rate="10" min_range="0.01" max_range="2.55" field_of_view="${30*M_PI/180}" ray_count="3">
     <origin xyz="0.0 0.0 ${SONAR_HEIGHT}" rpy="0 0 -0.785"/>
   </xacro:sonar_sensor>
-  <xacro:sonar_sensor name="sonar_sensor_five" parent="base_link" ros_topic="sonar_five" update_rate="10" min_range="0.01" max_range="3.0" field_of_view="${30*M_PI/180}" ray_count="3">
+  <xacro:sonar_sensor name="sonar_sensor_five" parent="base_link" ros_topic="sonar_5" update_rate="10" min_range="0.01" max_range="2.55" field_of_view="${30*M_PI/180}" ray_count="3">
     <origin xyz="0.0 0.0 ${SONAR_HEIGHT}" rpy="0 0 -1.309"/>
   </xacro:sonar_sensor>
-  <xacro:sonar_sensor name="sonar_sensor_six" parent="base_link" ros_topic="sonar_six" update_rate="10" min_range="0.01" max_range="3.0" field_of_view="${30*M_PI/180}" ray_count="3">
+  <xacro:sonar_sensor name="sonar_sensor_six" parent="base_link" ros_topic="sonar_6" update_rate="10" min_range="0.01" max_range="2.55" field_of_view="${30*M_PI/180}" ray_count="3">
     <origin xyz="0.0 0.0 ${SONAR_HEIGHT}" rpy="0 0 -1.833"/>
   </xacro:sonar_sensor>
-  <xacro:sonar_sensor name="sonar_sensor_seven" parent="base_link" ros_topic="sonar_seven" update_rate="10" min_range="0.01" max_range="3.0" field_of_view="${30*M_PI/180}" ray_count="3">
+  <xacro:sonar_sensor name="sonar_sensor_seven" parent="base_link" ros_topic="sonar_7" update_rate="10" min_range="0.01" max_range="2.55" field_of_view="${30*M_PI/180}" ray_count="3">
     <origin xyz="0.0 0.0 ${SONAR_HEIGHT}" rpy="0 0 -2.356"/>
   </xacro:sonar_sensor>
-  <xacro:sonar_sensor name="sonar_sensor_eight" parent="base_link" ros_topic="sonar_eight" update_rate="10" min_range="0.01" max_range="3.0" field_of_view="${30*M_PI/180}" ray_count="3">
+  <xacro:sonar_sensor name="sonar_sensor_eight" parent="base_link" ros_topic="sonar_8" update_rate="10" min_range="0.01" max_range="2.55" field_of_view="${30*M_PI/180}" ray_count="3">
     <origin xyz="0.0 0.0 ${SONAR_HEIGHT}" rpy="0 0 -2.88"/>
   </xacro:sonar_sensor>
-  <xacro:sonar_sensor name="sonar_sensor_nine" parent="base_link" ros_topic="sonar_nine" update_rate="10" min_range="0.01" max_range="3.0" field_of_view="${30*M_PI/180}" ray_count="3">
+  <xacro:sonar_sensor name="sonar_sensor_nine" parent="base_link" ros_topic="sonar_9" update_rate="10" min_range="0.01" max_range="2.55" field_of_view="${30*M_PI/180}" ray_count="3">
     <origin xyz="0.0 0.0 ${SONAR_HEIGHT}" rpy="0 0 2.88"/>
   </xacro:sonar_sensor>
-  <xacro:sonar_sensor name="sonar_sensor_ten" parent="base_link" ros_topic="sonar_ten" update_rate="10" min_range="0.01" max_range="3.0" field_of_view="${30*M_PI/180}" ray_count="3">
+  <xacro:sonar_sensor name="sonar_sensor_ten" parent="base_link" ros_topic="sonar_10" update_rate="10" min_range="0.01" max_range="2.55" field_of_view="${30*M_PI/180}" ray_count="3">
     <origin xyz="0.0 0.0 ${SONAR_HEIGHT}" rpy="0 0 2.356"/>
   </xacro:sonar_sensor>
-  <xacro:sonar_sensor name="sonar_sensor_eleven" parent="base_link" ros_topic="sonar_eleven" update_rate="10" min_range="0.01" max_range="3.0" field_of_view="${30*M_PI/180}" ray_count="3">
+  <xacro:sonar_sensor name="sonar_sensor_eleven" parent="base_link" ros_topic="sonar_11" update_rate="10" min_range="0.01" max_range="2.55" field_of_view="${30*M_PI/180}" ray_count="3">
     <origin xyz="0.0 0.0 ${SONAR_HEIGHT}" rpy="0 0 1.833"/>
   </xacro:sonar_sensor>
